File: charging_h-bridge.kicad_sch (KiCad schematic)
At the start: 10 parts, among them Q1 Q_PMOS_DGS, Q2 Q_NMOS_DGS, Q3 Q_PMOS_DGS, Q4 Q_NMOS_DGS

Commit message: More clean up
Connections:
- net +3V3: now also Q3.3 (S)
Changed lines of the file:
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@@
     (pin "1")
   )
-  (symbol (lib_id "power:+3.3V") (at 171.45 82.55 0) (unit 1)
+  (symbol (lib_id "power:+3.3V") (at 171.45 80.01 0) (unit 1)
     (in_bom yes) (on_board yes) (fields_autoplaced)
-    (property "Reference" "#PWR079" (id 0) (at 171.45 86.36 0)
+    (property "Reference" "#PWR079" (id 0) (at 171.45 83.82 0)
       (effects (font (size 1.27 1.27)) hide)
     )
-    (property "Value" "+3.3V" (id 1) (at 171.45 78.9455 0))
-    (property "Footprint" "" (id 2) (at 171.45 82.55 0)
+    (property "Value" "+3.3V" (id 1) (at 171.45 76.4055 0))
+    (property "Footprint" "" (id 2) (at 171.45 80.01 0)
       (effects (font (size 1.27 1.27)) hide)
     )
-    (property "Datasheet" "" (id 3) (at 171.45 82.55 0)
+    (property "Datasheet" "" (id 3) (at 171.45 80.01 0)
       (effects (font (size 1.27 1.27)) hide)
     )
